File: hotfire-board/Hotfire-Board/Hotfire-Board.kicad_pcb (KiCad board)
At the start: 2 copper layers, 85 parts, among them J1 Conn_01x02, J2 BCS-103-L-D-TE, J3 Conn_01x03, J4 Conn_01x03, J5 Conn_01x03, J6 USB4105-GF-A-060, J7 Conn_01x03, SW1 RESET, SW2 PTS526 SM15 SMTR2 LFS, U1 LMR36006BRNXR, U2 LMR36006CRNXT, U3 STM32L496RGT6, U4 TPS2113APW, U5 LP5912-3.3DRVR, U6 MAX31856MUD+, Y1 16MHz

Commit message: finished layout
Parts:
- added C43: 1u, Capacitor_SMD:C_0603_1608Metric, F.Cu at (145.2, 82.3)
- added C44: 0.1u, Capacitor_SMD:C_0402_1005Metric, F.Cu at (144.6, 81.1)
- added C45: 0.1u, Capacitor_SMD:C_0402_1005Metric, F.Cu at (164.9, 83.3)
- added C46: 0.1u, Capacitor_SMD:C_0402_1005Metric, F.Cu at (169.7, 83.3)
- added C47: 0.1u, Capacitor_SMD:C_0402_1005Metric, F.Cu at (166.2, 83.3)
- added C48: 0.1u, Capacitor_SMD:C_0402_1005Metric, F.Cu at (147.5, 107.6)
- added C49: 0.1u, Capacitor_SMD:C_0402_1005Metric, F.Cu at (155.3, 107.6)
- added C50: 0.1u, Capacitor_SMD:C_0402_1005Metric, F.Cu at (161.9, 107.6)
- added C51: 0.1u, Capacitor_SMD:C_0402_1005Metric, F.Cu at (170.3, 107.6)
- added C52: 0.1u, Capacitor_SMD:C_0402_1005Metric, F.Cu at (148.5, 98.6)
- added C53: 0.1u, Capacitor_SMD:C_0402_1005Metric, F.Cu at (156.8, 99.1)
- added C54: 0.1u, Capacitor_SMD:C_0402_1005Metric, F.Cu at (162.8, 98.8)
- added C55: 0.1u, Capacitor_SMD:C_0402_1005Metric, F.Cu at (172.0, 99.8)
- added C56: 10n, Capacitor_SMD:C_0402_1005Metric, F.Cu at (142.6, 109.0)
- added C57: 10n, Capacitor_SMD:C_0402_1005Metric, F.Cu at (147.6, 109.1)
- added C58: 10n, Capacitor_SMD:C_0402_1005Metric, F.Cu at (150.5, 109.0)
- added C59: 10n, Capacitor_SMD:C_0402_1005Metric, F.Cu at (155.3, 109.0)
- added C60: 0.1u, Capacitor_SMD:C_0402_1005Metric, F.Cu at (145.0, 108.3)
- added C61: 0.1u, Capacitor_SMD:C_0402_1005Metric, F.Cu at (152.9, 108.5)
- added C62: 10n, Capacitor_SMD:C_0402_1005Metric, F.Cu at (157.6, 109.0)
- added C63: 10n, Capacitor_SMD:C_0402_1005Metric, F.Cu at (162.4, 109.1)
- added C64: 10n, Capacitor_SMD:C_0402_1005Metric, F.Cu at (165.1, 109.0)
- added C65: 10n, Capacitor_SMD:C_0402_1005Metric, F.Cu at (169.9, 109.0)
- added C66: 0.1u, Capacitor_SMD:C_0402_1005Metric, F.Cu at (160.0, 108.1)
- added C67: 0.1u, Capacitor_SMD:C_0402_1005Metric, F.Cu at (167.5, 108.3)
- added C68: 0.1u, Capacitor_SMD:C_0402_1005Metric, F.Cu at (167.9, 83.3)
- added C69: 10u, Capacitor_SMD:C_1210_3225Metric, F.Cu at (199.5, 103.5)
- added C70: 10u, Capacitor_SMD:C_1210_3225Metric, F.Cu at (199.5, 110.4)
- added C71: 10u, Capacitor_SMD:C_1210_3225Metric, F.Cu at (189.9, 93.6)
- added CR6: SP1233-01ETG, MyFootprints:TVS_Input, F.Cu at (165.6, 92.4)
- added CR7: SP1233-01ETG, MyFootprints:TVS_Input, F.Cu at (180.8, 93.8)
- added CR8: SP1233-01ETG, MyFootprints:TVS_Input, F.Cu at (170.1, 92.2)
- added CR9: SP1233-01ETG, MyFootprints:TVS_Input, F.Cu at (175.1, 91.2)
- added D1: TPD1E05U06DPYR, MyFootprints:SD_ESD, F.Cu at (155.5, 75.3)
- added D10: BAT54S, MyFootprints:dual_shottkey, F.Cu at (171.7, 86.7)
- added D11: BAT54S, MyFootprints:dual_shottkey, F.Cu at (176.6, 85.2)
- added D12: TPD1E05U06DPYR, MyFootprints:SD_ESD, F.Cu at (210.0, 104.9)
- added D13: TPD1E05U06DPYR, MyFootprints:SD_ESD, F.Cu at (200.5, 106.9)
- added D14: TPD1E05U06DPYR, MyFootprints:SD_ESD, F.Cu at (203.2, 104.9)
- added D15: TPD1E05U06DPYR, MyFootprints:SD_ESD, F.Cu at (203.6, 109.7)
- added D16: TPD1E05U06DPYR, MyFootprints:SD_ESD, F.Cu at (198.5, 107.0)
- added D17: TPD1E05U06DPYR, MyFootprints:SD_ESD, F.Cu at (209.8, 109.7)
- added D18: TPD1E05U06DPYR, MyFootprints:SD_ESD, F.Cu at (190.7, 76.3)
- added D19: TPD1E05U06DPYR, MyFootprints:SD_ESD, F.Cu at (190.7, 74.0)
- added D2: TPD1E05U06DPYR, MyFootprints:SD_ESD, F.Cu at (152.8, 81.7)
- added D20: TPD1E05U06DPYR, MyFootprints:SD_ESD, F.Cu at (190.1, 91.4)
- added D21: TPD1E05U06DPYR, MyFootprints:SD_ESD, F.Cu at (190.7, 79.0)
- added D22: TPD1E05U06DPYR, MyFootprints:SD_ESD, F.Cu at (190.7, 83.9)
- added D23: TPD1E05U06DPYR, MyFootprints:SD_ESD, F.Cu at (190.7, 86.7)
- added D3: TPD1E05U06DPYR, MyFootprints:SD_ESD, F.Cu at (167.1, 63.7)
- added D4: TPD1E05U06DPYR, MyFootprints:SD_ESD, F.Cu at (164.0, 63.7)
- added D5: TPD1E05U06DPYR, MyFootprints:SD_ESD, F.Cu at (155.5, 71.2)
- added D6: BAT54S, MyFootprints:dual_shottkey, F.Cu at (166.4, 86.7)
- added D7: BAT54S, MyFootprints:dual_shottkey, F.Cu at (182.4, 88.6)
- added D8: TPD1E05U06DPYR, MyFootprints:SD_ESD, F.Cu at (155.5, 65.0)
- added D9: TPD1E05U06DPYR, MyFootprints:SD_ESD, F.Cu at (155.5, 68.1)
- added H1: MountingHole, MountingHole:MountingHole_3.2mm_M3, F.Cu at (210.3, 49.7)
- added H2: MountingHole, MountingHole:MountingHole_3.2mm_M3, F.Cu at (138.9, 113.8)
- added H3: MountingHole, MountingHole:MountingHole_3.2mm_M3, F.Cu at (210.3, 113.8)
- added H4: MountingHole, MountingHole:MountingHole_3.2mm_M3, F.Cu at (138.9, 49.7)
- added J10: Conn_01x03, Connector_Wire:SolderWire-0.5sqmm_1x03_P4.6mm_D0.9mm_OD2.1mm_Relief, F.Cu at (198.8, 98.9)
- added J11: 1725656, MyFootprints:screw_terminal, F.Cu at (143.6, 116.5)
- added J12: 1725656, MyFootprints:screw_terminal, F.Cu at (149.7, 116.5)
- added J13: 1725656, MyFootprints:screw_terminal, F.Cu at (155.8, 116.5)
- added J14: 1725656, MyFootprints:screw_terminal, F.Cu at (161.9, 116.5)
- added J15: Conn_01x08, Connector_PinSocket_2.54mm:PinSocket_1x08_P2.54mm_Vertical, F.Cu at (193.6, 72.2)
- added J8: MEM2061-01-188-00-A_REVA, MyFootprints:SD_Card, F.Cu at (144.6, 72.8)
- added J9: Conn_01x03, Connector_Wire:SolderWire-0.5sqmm_1x03_P4.6mm_D0.9mm_OD2.1mm_Relief, F.Cu at (186.8, 102.3)
- added R16: 22, Resistor_SMD:R_0402_1005Metric, F.Cu at (166.1, 63.8)
- added R17: 22, Resistor_SMD:R_0402_1005Metric, F.Cu at (162.9, 63.8)
- added R18: 22, Resistor_SMD:R_0402_1005Metric, F.Cu at (155.6, 66.1)
- added R19: 22, Resistor_SMD:R_0402_1005Metric, F.Cu at (155.6, 69.2)
- added R20: 22, Resistor_SMD:R_0402_1005Metric, F.Cu at (155.6, 73.3)
- added R21: 22, Resistor_SMD:R_0402_1005Metric, F.Cu at (155.6, 72.3)
- added R22: 47k, Resistor_SMD:R_0402_1005Metric, F.Cu at (155.6, 74.3)
- added R23: 47k, Resistor_SMD:R_0402_1005Metric, F.Cu at (151.7, 81.5)
- added R24: 47k, Resistor_SMD:R_0402_1005Metric, F.Cu at (168.2, 63.8)
- added R25: 20, Resistor_SMD:R_1206_3216Metric, F.Cu at (167.6, 92.7)
- added R26: 20, Resistor_SMD:R_1206_3216Metric, F.Cu at (183.6, 94.6)
- added R27: 47k, Resistor_SMD:R_0402_1005Metric, F.Cu at (165.1, 63.8)
- added R28: 130, Resistor_SMD:R_0805_2012Metric, F.Cu at (165.6, 89.4)
- added R29: 130, Resistor_SMD:R_0805_2012Metric, F.Cu at (182.0, 91.3)
- added R30: 4.7k, Resistor_SMD:R_0402_1005Metric, F.Cu at (167.8, 89.3)
- added R31: 4.7k, Resistor_SMD:R_0402_1005Metric, F.Cu at (184.2, 91.3)
- added R32: 47k, Resistor_SMD:R_0402_1005Metric, F.Cu at (155.6, 67.0)
- added R33: 47k, Resistor_SMD:R_0402_1005Metric, F.Cu at (155.6, 70.2)
- added R34: 20, Resistor_SMD:R_1206_3216Metric, F.Cu at (172.4, 92.7)
- added R35: 130, Resistor_SMD:R_0805_2012Metric, F.Cu at (170.8, 89.5)
- added R36: 4.7k, Resistor_SMD:R_0402_1005Metric, F.Cu at (173.0, 89.4)
- added R37: 10k, Resistor_SMD:R_0402_1005Metric, F.Cu at (146.8, 98.2)
- added R38: 10k, Resistor_SMD:R_0402_1005Metric, F.Cu at (155.0, 98.2)
- added R39: 10k, Resistor_SMD:R_0402_1005Metric, F.Cu at (161.5, 98.1)
- added R40: 10k, Resistor_SMD:R_0402_1005Metric, F.Cu at (169.5, 98.3)
- added R41: 20, Resistor_SMD:R_1206_3216Metric, F.Cu at (177.5, 91.2)
- added R42: 130, Resistor_SMD:R_0805_2012Metric, F.Cu at (176.0, 87.9)
- added R43: 4.7k, Resistor_SMD:R_0402_1005Metric, F.Cu at (178.2, 87.9)
- added R44: 100, Resistor_SMD:R_0402_1005Metric, F.Cu at (143.6, 109.0)
- added R45: 100, Resistor_SMD:R_0402_1005Metric, F.Cu at (146.4, 109.0)
- added R46: 100, Resistor_SMD:R_0402_1005Metric, F.Cu at (151.4, 109.0)
- added R47: 100, Resistor_SMD:R_0402_1005Metric, F.Cu at (154.3, 109.0)
- added R48: 100, Resistor_SMD:R_0402_1005Metric, F.Cu at (158.6, 109.0)
- added R49: 100, Resistor_SMD:R_0402_1005Metric, F.Cu at (161.4, 109.1)
- added R50: 100, Resistor_SMD:R_0402_1005Metric, F.Cu at (166.1, 109.0)
- added R51: 100, Resistor_SMD:R_0402_1005Metric, F.Cu at (168.9, 109.0)
- added R52: 100, Resistor_SMD:R_0402_1005Metric, F.Cu at (208.0, 104.9)
- added R53: 100, Resistor_SMD:R_0402_1005Metric, F.Cu at (205.2, 104.9)
- added R54: 100, Resistor_SMD:R_0402_1005Metric, F.Cu at (205.7, 109.6)
- added R55: 100, Resistor_SMD:R_0402_1005Metric, F.Cu at (207.7, 109.6)
- added R56: 100, Resistor_SMD:R_0402_1005Metric, F.Cu at (190.8, 77.4)
- added R57: 100, Resistor_SMD:R_0402_1005Metric, F.Cu at (190.8, 75.1)
- added R58: 100, Resistor_SMD:R_0402_1005Metric, F.Cu at (190.8, 80.1)
- added R59: 100, Resistor_SMD:R_0402_1005Metric, F.Cu at (190.8, 85.0)
- added R60: 100, Resistor_SMD:R_0402_1005Metric, F.Cu at (190.8, 87.7)
- added U7: MAX31856MUD+, MyFootprints:MAX, F.Cu at (153.2, 103.2)
- added U8: MAX31856MUD+, MyFootprints:MAX, F.Cu at (159.9, 103.0)
- added U9: MAX31856MUD+, MyFootprints:MAX, F.Cu at (167.9, 103.2)
- J3: value Conn_01x03 -> UART1; footprint Connector_Wire:SolderWire-0.5sqmm_1x03_P4.6mm_D0.9mm_OD2.1mm_Relief -> Connector_PinSocket_2.54mm:PinSocket_1x04_P2.54mm_Vertical
- J4: value Conn_01x03 -> UART3; footprint Connector_Wire:SolderWire-0.5sqmm_1x03_P4.6mm_D0.9mm_OD2.1mm_Relief -> Connector_PinSocket_2.54mm:PinSocket_1x04_P2.54mm_Vertical
- SW2: value PTS526 SM15 SMTR2 LFS -> BOOT
- moved J1 108.2 mm to (200.3, 48.7), turned to -90 degrees
- moved CR1 81.8 mm to (191.9, 57.0)
- moved CR2 77.1 mm to (187.9, 64.6), turned to -90 degrees
- moved J3 74.5 mm to (211.5, 102.5), turned to -90 degrees
- moved R8 69.8 mm to (210.9, 56.0)
- moved J4 66.7 mm to (211.5, 107.3), turned to -90 degrees
- moved R15 63.7 mm to (144.6, 49.5), turned to 90 degrees
- moved F1 62.3 mm to (198.5, 57.0), turned to 180 degrees
- moved C6 62.2 mm to (204.6, 58.0)
- moved U5 61.0 mm to (151.5, 54.9), turned to 180 degrees
- moved LED4 60.1 mm to (143.6, 52.4), turned to 180 degrees
- moved R11 59.4 mm to (158.2, 47.2), turned to 180 degrees
- moved C32 57.4 mm to (151.3, 50.5), turned to -90 degrees
- moved C28 56.6 mm to (169.1, 51.2), turned to -90 degrees
- moved U1 56.6 mm to (173.0, 60.5)
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Connections:
- net Net-(CR1-Pad2) renamed BAT_FUSE
- net Net-(J1-Pin_2) renamed BAT_IN
- net Net-(U1-NC) renamed SW
- net Net-(U2-NC) renamed SW1
- C17 pad 2: AGND -> GND
- C26 pad 2: Net-(C26-Pad2) -> /NRST
- C29 pad 2: 3V3_BUCK -> 3V3_LDO
- C30 pad 1: 3V3_LDO -> 3V3_BUCK
- CR3 pad 2: PGND -> GND
- J3 pad 1: 15V0 -> GND
- J3 pad 2: GND -> Net-(D12-I/O)
- J3 pad 3: /Pressure_1 -> Net-(D14-I/O)
- J4 pad 1: 15V0 -> GND
- J4 pad 2: GND -> Net-(D17-I/O)
- J4 pad 3: /Pressure_2 -> Net-(D15-I/O)
- J5 pad 3: /Pressure_3 -> Net-(J5-Pin_3)
- J6 pad A1_B12: PGND -> GND
- J6 pad B1_A12: PGND -> GND
- J6 pad SH1: PGND -> GND
- J6 pad SH2: PGND -> GND
- J6 pad SH3: PGND -> GND
- J6 pad SH4: PGND -> GND
- J7 pad 3: /Pressure_4 -> Net-(J7-Pin_3)
- R10 pad 2: 3V3_BUCK -> 3V3_LDO
- R11 pad 1: 3V3_LDO -> 3V3_BUCK
- R9 pad 2: Net-(C26-Pad2) -> /NRST
- SW1 pad 1: Net-(C26-Pad2) -> /NRST
- SW1 pad 2: Net-(C26-Pad2) -> /NRST
- U3 pad 10: unconnected-(U3A-PC2-Pad10) -> /P2
- U3 pad 11: unconnected-(U3A-PC3-Pad11) -> /P3
- U3 pad 21: unconnected-(U3A-PA5-Pad21) -> /CS1
- U3 pad 22: unconnected-(U3A-PA6-Pad22) -> /CS2
- U3 pad 23: unconnected-(U3A-PA7-Pad23) -> /CS3
- U3 pad 24: unconnected-(U3A-PC4-Pad24) -> /CS4
- U3 pad 25: unconnected-(U3A-PC5-Pad25) -> /GPIO_OUT_1
- U3 pad 26: unconnected-(U3A-PB0-Pad26) -> /GPIO_OUT_0
- U3 pad 29: unconnected-(U3A-PB10-Pad29) -> /TX3
- U3 pad 30: unconnected-(U3A-PB11-Pad30) -> /RX3
- U3 pad 34: unconnected-(U3A-PB13-Pad34) -> /CLK
- U3 pad 35: unconnected-(U3A-PB14-Pad35) -> /MISO
- U3 pad 36: unconnected-(U3A-PB15-Pad36) -> /MOSI
- U3 pad 38: unconnected-(U3A-PC7-Pad38) -> /SD_DET
- U3 pad 39: unconnected-(U3A-PC8-Pad39) -> /SD_D0
- U3 pad 40: unconnected-(U3A-PC9-Pad40) -> /SD_D1
- U3 pad 42: unconnected-(U3A-PA9-Pad42) -> /TX1
- U3 pad 43: unconnected-(U3A-PA10-Pad43) -> /RX1
- U3 pad 51: unconnected-(U3A-PC10-Pad51) -> /SD_D2
- U3 pad 52: unconnected-(U3A-PC11-Pad52) -> /SD_D3
- U3 pad 53: unconnected-(U3A-PC12-Pad53) -> /SD_CLK
- U3 pad 54: unconnected-(U3A-PD2-Pad54) -> /SD_CMD
- U3 pad 8: unconnected-(U3A-PC0-Pad8) -> /P0
- U3 pad 9: unconnected-(U3A-PC1-Pad9) -> /P1
- U4 pad 6: 3V3_LDO -> 3V3_BUCK
- U4 pad 8: 3V3_BUCK -> 3V3_LDO
- U5 pad 5: AGND -> GND
- U5 pad 7: AGND -> GND
- U5 pad 8: AGND -> GND
- U5 pad 9: (no net) -> GND
- U6 pad 1: unconnected-(U6-AGND-Pad1) -> GND
- U6 pad 10: unconnected-(U6-SCK-Pad10) -> /CLK
- U6 pad 11: unconnected-(U6-SDO-Pad11) -> /MISO
- U6 pad 12: unconnected-(U6-SDI-Pad12) -> /MOSI
- U6 pad 14: unconnected-(U6-DGND-Pad14) -> GND
- U6 pad 2: unconnected-(U6-BIAS-Pad2) -> Net-(U6-BIAS)
- U6 pad 3: unconnected-(U6-T--Pad3) -> Net-(U6-T-)
- U6 pad 4: unconnected-(U6-T+-Pad4) -> Net-(U6-T+)
- U6 pad 5: unconnected-(U6-AVDD-Pad5) -> 3V3
- U6 pad 8: unconnected-(U6-DVDD-Pad8) -> 3V3
- U6 pad 9: unconnected-(U6-*CS-Pad9) -> /CS1
Routing:
- net 3V3: track 0.00 -> 180.7 mm, vias 0 -> 52
- net 15V0: track 0.00 -> 117.8 mm, vias 0 -> 7
- net /MOSI: track 0.00 -> 97.1 mm, vias 0 -> 5
- net /MISO: track 0.00 -> 93.9 mm, vias 0 -> 5
- net /CLK: track 0.00 -> 90.9 mm, vias 0 -> 5
- net /RX1: track 0.00 -> 83.7 mm, vias 0 -> 2
- net /TX1: track 0.00 -> 75.5 mm, vias 0 -> 2
- net /TX3: track 0.00 -> 68.6 mm, vias 0 -> 2
- net /RX3: track 0.00 -> 64.6 mm, vias 0 -> 2
- net /SWCLK: track 0.00 -> 57.2 mm, vias 0 -> 1
- net /CS1: track 0.00 -> 55.9 mm, vias 0 -> 2
- net GND: track 0.00 -> 54.7 mm, vias 0 -> 252
- net /SWDIO: track 0.00 -> 52.9 mm, vias 0 -> 1
- net /NRST: track 0.00 -> 48.3 mm, vias 0 -> 1
- net /SWO: track 0.00 -> 47.6 mm, vias 0 -> 1
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- added copper zone on F.Cu, net 15V0
- added copper zone on F.Cu, net 3V3
- added copper zone on In2.Cu, net 3V3
- added copper zone on F.Cu, net 3V3_BUCK
- added copper zone on F.Cu, net 3V3_LDO
- added copper zone on F.Cu, net BAT_FUSE
- added copper zone on F.Cu, net BAT_IN
- added copper zone on B.Cu, net GND
- added copper zone on F.Cu, net GND
- added copper zone on In1.Cu, net GND
- added copper zone on In2.Cu, net GND
- added copper zone on F.Cu, net SW
- added copper zone on F.Cu, net SW1
- added copper zone on F.Cu, net VBAT
- added copper zone on In1.Cu, net VBAT
- added copper zone on In2.Cu, net VBAT
Other:
- board outline added: 78.4 x 71 mm
- copper layers 2 -> 4
- board text added: "+"
- board text added: "-"
- board text added: "15V0"
- board text added: "3V3"
- board text added: "3V3 Buck"
- board text added: "3V3 LDO"
- board text added: "BOOT"
- board text added: "CLK"
- board text added: "GND"
- board text added: "GPIO"
- board text added: "Gaucho Rocket Project 26-27 Data Logger Board By: Andrew Liu"
- board text added: "MISO"
- board text added: "MOSI"
- board text added: "NRST"
- board text added: "RESET"
- board text added: "RX"
- board text added: "SWCLK"
- board text added: "SWD"
- board text added: "SWDIO"
- board text added: "SWO"
- board text added: "TX"
- board text added: "UART1"
- board text added: "UART3"

Commit message: order read
Parts:
- added LED5: LTST-C190KRKT, MyFootprints:red_LED, F.Cu at (174.3, 69.1)
- added R61: 130, Resistor_SMD:R_0805_2012Metric, F.Cu at (175.2, 70.9)
- moved R57 2.47 mm to (188.3, 75.0)
- moved D19 2.46 mm to (188.2, 73.9)
- moved D23 2.40 mm to (188.3, 86.5)
- moved R60 2.40 mm to (188.4, 87.6)
- moved D22 2.40 mm to (188.3, 83.7)
- moved R59 2.40 mm to (188.4, 84.8)
- moved D18 2.37 mm to (188.3, 76.3)
- moved R56 2.37 mm to (188.4, 77.4)
- moved D21 2.36 mm to (188.3, 79.2)
- moved R58 2.36 mm to (188.4, 80.3)
- moved C71 1.63 mm to (188.2, 93.6)
- moved D20 1.31 mm to (188.8, 91.4)
- moved C54 0.44 mm to (163.3, 98.7)
- moved C45 0.32 mm to (164.8, 83.0)
Connections:
- U3 pad 27: unconnected-(U3A-PB1-Pad27) -> /STATUS_LED
Routing:
- net Net-(D19-I/O): track 5.11 -> 10.0 mm
- net Net-(D22-I/O): track 5.10 -> 9.98 mm
- net Net-(D23-I/O): track 5.11 -> 9.91 mm
- net Net-(D18-I/O): track 5.14 -> 9.87 mm
- net Net-(D21-I/O): track 5.13 -> 9.83 mm
- net /STATUS_LED: track 0.00 -> 4.10 mm
- net /MOSI: track 97.1 -> 93.3 mm
- net Net-(LED5-Pad2): track 0.00 -> 3.28 mm
- net 3V3: track 180.7 -> 183.8 mm
- net /MISO: track 93.9 -> 91.6 mm
- net /CLK: track 90.9 -> 89.2 mm
- net GND: track 54.7 -> 53.4 mm
- net /GPIO_OUT_0: track 25.2 -> 24.5 mm
- net /GPIO_OUT_1: track 26.5 -> 25.7 mm

Commit message: reworked power poath, added cs multiplexer
Parts:
- removed CR2: SMBJ28A-13-F, MyFootprints:28V_TVS
- added C72: 4.7u, Capacitor_SMD:C_1206_3216Metric, F.Cu at (209.1, 67.2)
- added C73: 4.7u, Capacitor_SMD:C_1206_3216Metric, F.Cu at (209.1, 64.9)
- added C74: 0.1u, Capacitor_SMD:C_0402_1005Metric, F.Cu at (212.6, 74.8)
- added C75: 0.1u, Capacitor_SMD:C_0402_1005Metric, F.Cu at (206.8, 84.6)
- added C76: 0.1u, Capacitor_SMD:C_0402_1005Metric, F.Cu at (211.3, 83.6)
- added C77: 4.7u, Capacitor_SMD:C_1206_3216Metric, F.Cu at (210.4, 85.3)
- added C78: 0.1u, Capacitor_SMD:C_0402_1005Metric, F.Cu at (207.1, 74.4)
- added C79: 0.1u, Capacitor_SMD:C_0402_1005Metric, F.Cu at (180.3, 73.5)
- added C80: 1u, Capacitor_SMD:C_0603_1608Metric, F.Cu at (180.0, 72.2)
- added D24: SMBJ15A, MyFootprints:15V_TVS, F.Cu at (186.8, 58.0)
- added D25: SMBJ18A, MyFootprints:18V_TVS, F.Cu at (206.4, 97.8)
- added D26: TPD1E05U06DPYR, MyFootprints:SD_ESD, F.Cu at (190.4, 89.6)
- added D27: TPD1E05U06DPYR, MyFootprints:SD_ESD, F.Cu at (190.4, 97.9)
- added D28: TPD1E05U06DPYR, MyFootprints:SD_ESD, F.Cu at (192.5, 89.6)
- added D29: TPD1E05U06DPYR, MyFootprints:SD_ESD, F.Cu at (181.8, 89.6)
- added D30: TPD1E05U06DPYR, MyFootprints:SD_ESD, F.Cu at (181.8, 97.9)
- added D31: TPD1E05U06DPYR, MyFootprints:SD_ESD, F.Cu at (184.0, 89.6)
- added D32: TPD1E05U06DPYR, MyFootprints:SD_ESD, F.Cu at (184.0, 97.9)
- added D33: TPD1E05U06DPYR, MyFootprints:SD_ESD, F.Cu at (186.1, 89.6)
- added D34: TPD1E05U06DPYR, MyFootprints:SD_ESD, F.Cu at (186.1, 97.9)
- added D35: TPD1E05U06DPYR, MyFootprints:SD_ESD, F.Cu at (188.2, 89.6)
- added D36: TPD1E05U06DPYR, MyFootprints:SD_ESD, F.Cu at (188.2, 97.9)
- added J16: C36191, Connector_PinSocket_2.54mm:PinSocket_2x06_P2.54mm_Vertical, F.Cu at (182.1, 92.5)
- added LED6: LTST-C190KRKT, MyFootprints:red_LED, F.Cu at (150.8, 56.2)
- added R62: 68.1k, Resistor_SMD:R_0402_1005Metric, F.Cu at (205.6, 74.4)
- added R63: 10k, Resistor_SMD:R_0402_1005Metric, F.Cu at (205.1, 75.8)
- added R64: 68.1k, Resistor_SMD:R_0402_1005Metric, F.Cu at (206.3, 71.1)
- added R65: 100k, Resistor_SMD:R_0402_1005Metric, F.Cu at (210.7, 74.6)
- added R66: 100k, Resistor_SMD:R_0402_1005Metric, F.Cu at (210.7, 73.6)
- added R67: 4.7k, Resistor_SMD:R_0402_1005Metric, F.Cu at (210.7, 72.6)
- added R68: 590, Resistor_SMD:R_0402_1005Metric, F.Cu at (210.7, 71.6)
- added R69: 10k, Resistor_SMD:R_0402_1005Metric, F.Cu at (208.8, 72.2)
- added R70: 4.7k, Resistor_SMD:R_0402_1005Metric, F.Cu at (208.0, 71.2)
- added R71: 130, Resistor_SMD:R_0805_2012Metric, F.Cu at (168.1, 50.6)
- added R72: 10k, Resistor_SMD:R_0402_1005Metric, F.Cu at (206.8, 83.7)
- added R73: 4.7k, Resistor_SMD:R_0402_1005Metric, F.Cu at (205.3, 83.2)
- added R74: 100k, Resistor_SMD:R_0402_1005Metric, F.Cu at (208.1, 74.3)
- added R75: 10k, Resistor_SMD:R_0402_1005Metric, F.Cu at (182.5, 71.9)
- added R76: 10k, Resistor_SMD:R_0402_1005Metric, F.Cu at (186.6, 71.9)
- added R77: 10k, Resistor_SMD:R_0402_1005Metric, F.Cu at (183.9, 71.9)
- added R78: 10k, Resistor_SMD:R_0402_1005Metric, F.Cu at (185.3, 71.9)
- added R79: 130, Resistor_SMD:R_0805_2012Metric, F.Cu at (158.7, 50.8)
- added R80: 100, Resistor_SMD:R_0402_1005Metric, F.Cu at (180.7, 89.7)
- added R81: 100, Resistor_SMD:R_0402_1005Metric, F.Cu at (182.9, 89.7)
- added R82: 100, Resistor_SMD:R_0402_1005Metric, F.Cu at (185.0, 89.7)
- added R83: 100, Resistor_SMD:R_0402_1005Metric, F.Cu at (187.2, 89.7)
- added R84: 100, Resistor_SMD:R_0402_1005Metric, F.Cu at (189.3, 89.7)
- added R85: 100, Resistor_SMD:R_0402_1005Metric, F.Cu at (191.4, 89.7)
- added R86: 100, Resistor_SMD:R_0402_1005Metric, F.Cu at (180.7, 97.8)
- added R87: 100, Resistor_SMD:R_0402_1005Metric, F.Cu at (182.9, 97.8)
- added R88: 100, Resistor_SMD:R_0402_1005Metric, F.Cu at (185.0, 97.8)
- added R89: 100, Resistor_SMD:R_0402_1005Metric, F.Cu at (187.2, 97.8)
- added R90: 100, Resistor_SMD:R_0402_1005Metric, F.Cu at (189.3, 97.8)
- added R91: 130, Resistor_SMD:R_0805_2012Metric, F.Cu at (152.7, 54.2)
- added R92: 130, Resistor_SMD:R_0805_2012Metric, F.Cu at (153.9, 56.1)
- added U10: SS34, MyFootprints:Boost_Shottkey, F.Cu at (203.7, 62.4)
- added U11: CD74HC154M96, MyFootprints:4-16-Multiplexer, F.Cu at (187.8, 80.0)
- added U12: TPS26600PWPR, MyFootprints:eFuse, F.Cu at (209.9, 79.2)
- C10: value 220n -> 10n; footprint Capacitor_SMD:C_0805_2012Metric -> Capacitor_SMD:C_0402_1005Metric
- C13: value 1u -> 270n; footprint Capacitor_SMD:C_0603_1608Metric -> Capacitor_SMD:C_0402_1005Metric
- C16: value 0.1u -> 100p
- C18: value CFF -> 0.1u; footprint Capacitor_SMD:C_0603_1608Metric -> Capacitor_SMD:C_0402_1005Metric
- C20: value 0.1u -> 4.7u; footprint Capacitor_SMD:C_0402_1005Metric -> Capacitor_SMD:C_1206_3216Metric
- C22, C24: value 10u -> 4.7u; footprint Capacitor_SMD:C_1210_3225Metric -> Capacitor_SMD:C_1206_3216Metric
- C9: value 220n -> 0.1u; footprint Capacitor_SMD:C_0805_2012Metric -> Capacitor_SMD:C_0402_1005Metric
- J1: footprint Connector_Wire:SolderWire-0.5sqmm_1x02_P4.6mm_D0.9mm_OD2.1mm_Relief -> Connector_AMASS:AMASS_XT60-F_1x02_P7.20mm_Vertical
- J10, J5, J7, J9: value Conn_01x03 -> SM03B-GHS-TB; footprint Connector_Wire:SolderWire-0.5sqmm_1x03_P4.6mm_D0.9mm_OD2.1mm_Relief -> MyFootprints:3-pin-jst
- L1, L2: value XAL4040-153MEC -> IHLP2525CZER220M5A; footprint MyFootprints:15uH_Inductor -> MyFootprints:22uH
- R2: value 100k -> 590
- R5: value 7.15k -> 43.2k
- R7: value 43.2k -> 24.9k
- U2: value LMR36006CRNXT -> TPS55340PWPR; footprint MyFootprints:15V_Buck -> MyFootprints:15V_Boost
- U3: value STM32L496RGT6 -> STM32L496RET6
- moved J4 73.8 mm to (137.7, 108.1), turned to 180 degrees
- moved D17 69.3 mm to (140.6, 105.8)
- moved R55 67.4 mm to (140.5, 104.7), turned to 0 degrees
- moved R54 65.5 mm to (140.5, 102.5)
- moved D15 63.3 mm to (140.6, 103.6), turned to 0 degrees
- moved D16 62.1 mm to (137.0, 98.1), turned to 180 degrees
- moved C70 59.3 mm to (141.2, 99.8), turned to -90 degrees
- moved J5 38.8 mm to (172.6, 113.8), turned to 0 degrees
- moved L2 32.8 mm to (178.4, 52.8), turned to -90 degrees
- moved R8 31.6 mm to (210.5, 87.6)
- moved LED2 31.4 mm to (207.4, 87.3), turned to -90 degrees
- moved J3 27.8 mm to (184.0, 106.8), turned to 90 degrees
- moved D22 27.3 mm to (208.9, 101.6)
- moved D20 27.1 mm to (208.9, 109.6)
- moved D23 26.9 mm to (208.9, 103.8)
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Connections:
- C1 pad 2: 5V0 -> 5V_USB
- C10 pad 1: GND -> Net-(U2-SS)
- C10 pad 2: VBAT -> GND
- C11 pad 1: 5V0 -> 5V_USB
- C13 pad 1: Net-(U2-VCC) -> Net-(C13-Pad1)
- C16 pad 1: Net-(U2-BST) -> Net-(U2-COMP)
- C16 pad 2: SW1 -> GND
- C17 pad 1: 3V3_LDO -> 3V3
- C18 pad 1: 15V0 -> 15V0_Boost
- C18 pad 2: Net-(U2-FB) -> GND
- C19 pad 1: 3V3_BUCK -> 5V_BUCK
- C20 pad 1: 15V0 -> 15V0_Boost
- C21 pad 1: 3V3_BUCK -> 5V_BUCK
- C22 pad 1: 15V0 -> 15V0_Boost
- C23 pad 1: 3V3_BUCK -> 5V_BUCK
- C24 pad 1: 15V0 -> 15V0_Boost
- C25 pad 1: 3V3_BUCK -> 5V_BUCK
- C27 pad 1: 3V3_BUCK -> 5V_BUCK
- C28 pad 1: 3V3_BUCK -> 5V_BUCK
- C29 pad 2: 3V3_LDO -> 5V_BUCK
- C30 pad 1: 3V3_BUCK -> 5V_USB
- C31 pad 1: 3V3 -> 5V0
- C32 pad 1: 3V3 -> 5V0
- C4 pad 1: 5V0 -> 5V_USB
- C9 pad 1: GND -> VBAT
- C9 pad 2: VBAT -> GND
- CR3 pad 5: 5V0 -> 5V_USB
- J5 pad 3: Net-(J5-Pin_3) -> Net-(J5-Pad3)
- J6 pad A4_B9: 5V0 -> 5V_USB
- J6 pad B4_A9: 5V0 -> 5V_USB
- J7 pad 3: Net-(J7-Pin_3) -> Net-(J7-Pad3)
- L1 pad 1: SW -> ANODE
- L1 pad 2: 3V3_BUCK -> VBAT
- L2 pad 1: SW1 -> 5V_BUCK
- L2 pad 2: 15V0 -> SW
- R1 pad 2: 3V3_LDO -> 3V3
- R10 pad 2: 3V3_LDO -> 5V_BUCK
- R11 pad 1: 3V3_BUCK -> 5V_USB
- R14 pad 2: 3V3_BUCK -> Net-(R14-Pad2)
- R15 pad 2: 3V3 -> Net-(R15-Pad2)
- R2 pad 1: 15V0 -> Net-(U2-COMP)
- R2 pad 2: Net-(U2-FB) -> Net-(C13-Pad1)
- R25 pad 2: Net-(J7-Pin_3) -> Net-(J5-Pad3)
- R26 pad 2: Net-(J5-Pin_3) -> Net-(J7-Pad3)
- R37 pad 2: /CS1 -> /CS0
- R38 pad 2: /CS2 -> /CS1
- R39 pad 2: /CS3 -> /CS2
- R40 pad 2: /CS4 -> /CS3
- R5 pad 1: Net-(U2-FB) -> 15V0_Boost
- R5 pad 2: GND -> Net-(R5-Pad2)
- R52 pad 2: /RX1 -> /TX1
- R53 pad 2: /TX1 -> /RX1
- R54 pad 2: /RX3 -> /TX3
- R55 pad 2: /TX3 -> /RX3
- R57 pad 2: /MOSI -> /CLK
- R58 pad 2: /CLK -> /MOSI
- R6 pad 1: 3V3_BUCK -> 5V_BUCK
- U2 pad 1: GND -> ANODE
- U2 pad 10: VBAT -> Net-(U2-FREQ)
- U2 pad 12: SW1 -> GND
- U2 pad 2: VBAT -> ANODE
- U2 pad 3: SW1 -> VBAT
- U2 pad 4: Net-(U2-BST) -> VBAT
- U2 pad 5: Net-(U2-VCC) -> Net-(U2-SS)
- U2 pad 7: Net-(U2-FB) -> GND
- U2 pad 8: unconnected-(U2-PG-Pad8) -> Net-(U2-COMP)
- U2 pad 9: VBAT -> Net-(U2-FB)
- U3 pad 21: /CS1 -> /A0
- U3 pad 22: /CS2 -> /A1
- U3 pad 23: /CS3 -> /A2
- U3 pad 24: /CS4 -> /A3
- U4 pad 6: 3V3_BUCK -> 5V_USB
- U4 pad 7: 3V3 -> 5V0
- U4 pad 8: 3V3_LDO -> 5V_BUCK
- U5 pad 1: 3V3_LDO -> 3V3
- U6 pad 9: /CS1 -> /CS0
- U7 pad 9: /CS2 -> /CS1
- U8 pad 9: /CS3 -> /CS2
- U9 pad 9: /CS4 -> /CS3
Routing:
- net /CS0: track 0.00 -> 57.2 mm, vias 0 -> 2
- net /CS14: track 0.00 -> 53.3 mm
- net /CS13: track 0.00 -> 48.4 mm
- net /MOSI: track 93.3 -> 140.8 mm, vias 5 -> 6
- net /CS12: track 0.00 -> 43.2 mm
- net /MISO: track 91.6 -> 133.9 mm, vias 5 -> 8
- net /CS4: track 47.5 -> 8.42 mm, vias 2 -> 0
- net /CLK: track 89.2 -> 126.8 mm, vias 5 -> 8
- net /CS11: track 0.00 -> 36.8 mm
- net /GPIO_OUT_1: track 25.7 -> 60.1 mm, vias 0 -> 2
- net 5V_USB: track 0.00 -> 33.7 mm
- net Net-(J5-Pin_3): track 33.0 -> 0.00 mm
- net /GPIO_OUT_0: track 24.5 -> 56.4 mm, vias 0 -> 2
- net Net-(J7-Pad3): track 0.00 -> 25.8 mm
- net /CS10: track 0.00 -> 25.3 mm
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- added copper zone on F.Cu, net 15V0_Boost
- added copper zone on F.Cu, net 5V0
- added copper zone on F.Cu, net 5V_BUCK
- added copper zone on F.Cu, net 5V_USB
- added copper zone on F.Cu, net ANODE
- removed copper zone on F.Cu, net 3V3_BUCK
- removed copper zone on F.Cu, net 3V3_LDO
- removed copper zone on F.Cu, net BAT_FUSE
- removed copper zone on F.Cu, net SW1
- removed copper zone on In2.Cu, net VBAT
Other:
- board size 78.4 x 71 mm -> 78.7 x 71 mm
- board text added: "10"
- board text added: "11"
- board text added: "12"
- board text added: "13"
- board text added: "14"
- board text added: "4"
- board text added: "5"
- board text added: "5V0"
- board text added: "5V0-Buck"
- board text added: "5V0_USB"
- board text added: "6"
- board text added: "7"
- board text added: "8"
- board text added: "9"
- board text added: "G"
- board text added: "IO1"
- board text added: "IO2"
- board text added: "SPI2"
- board text removed: "3V3 Buck"
- board text removed: "3V3 LDO"
- board text removed: "GPIO"
