File: hotfire-board/Hotfire-Board/Hotfire-Board.kicad_pcb (KiCad board)
At the start: 4 copper layers, 78.7 x 71 mm, 260 parts, among them J1 Conn_01x02, J10 SM03B-GHS-TB, J11 1725656, J12 1725656, J13 1725656, J14 1725656, J15 Conn_01x08, J16 C36191, J2 BCS-103-L-D-TE, J3 UART1, J4 UART3, J5 SM03B-GHS-TB, J6 USB4105-GF-A-060, J7 SM03B-GHS-TB, J8 MEM2061-01-188-00-A_REVA, J9 SM03B-GHS-TB, SW1 RESET, SW2 BOOT, U1 LMR36006BRNXR, U10 SS34, U11 CD74HC154M96, U12 TPS26600PWPR, U2 TPS55340PWPR, U3 STM32L496RET6, U4 TPS2113APW, U5 LP5912-3.3DRVR, U6 MAX31856MUD+, U7 MAX31856MUD+, U8 MAX31856MUD+, U9 MAX31856MUD+, Y1 16MHz

Commit message: prod ready
Parts:
- C69, C70, C71: value 10u -> 1u; footprint Capacitor_SMD:C_1210_3225Metric -> Capacitor_SMD:C_0603_1608Metric
- J1: footprint Connector_AMASS:AMASS_XT60-F_1x02_P7.20mm_Vertical -> Connector_AMASS:AMASS_XT60-M_1x02_P7.20mm_Vertical
- moved C69 1.05 mm to (195.0, 106.2)
- moved C70 0.56 mm to (141.1, 100.3), turned to 180 degrees
- moved C71 0.37 mm to (208.5, 107.0), turned to 0 degrees
- moved C41 0.27 mm to (158.6, 79.0)
Routing:
- net GND: vias 314 -> 345
