File: hotfire-board/Hotfire-Board/Hotfire-Board.kicad_sch (KiCad schematic)
At the start: 127 parts, among them J1 Conn_01x02, J2 BCS-103-L-D-TE, J3 Conn_01x03, J4 Conn_01x03, J5 Conn_01x03, J6 USB4105-GF-A-060, J7 Conn_01x03, SW1 RESET, SW2 PTS526 SM15 SMTR2 LFS, U1 LMR36006BRNXR, U2 LMR36006CRNXT, U3 STM32L496RGT6, U4 TPS2113APW, U5 LP5912-3.3DRVR, U6 MAX31856MUD+, Y1 16MHz

Commit message: finished layout
Parts:
- removed J3, J4: Conn_01x03, Connector_Wire:SolderWire-0.5sqmm_1x03_P4.6mm_D0.9mm_OD2.1mm_Relief, symbol Connector_Generic:Conn_01x03
- removed J?: UART1, Connector_PinSocket_2.54mm:PinSocket_1x03_P2.54mm_Vertical, symbol Connector_Generic:Conn_01x03
- removed J?: 1040310811, MyFootprints:SD_Module, symbol SD_Module:1040310811
- removed J?: UART3, Connector_PinSocket_2.54mm:PinSocket_1x04_P2.54mm_Vertical, symbol Connector_Generic:Conn_01x04
- added C43: 1u, Capacitor_SMD:C_0603_1608Metric, symbol Device:C
- added C44, C45, C46, C47, C68: 0.1u, Capacitor_SMD:C_0402_1005Metric, symbol Device:C
- added C69, C70, C71: 10u, Capacitor_SMD:C_1210_3225Metric, symbol Device:C
- added CR6, CR7, CR8, CR9: SP1233-01ETG, MyFootprints:TVS_Input, symbol TVS_Input:SP1233-01ETG
- added D1, D12, D13, D14, D15, D16, D17, D18, D19, D2, D20, D21, D22, D23, D3, D4, D5, D8, D9: TPD1E05U06DPYR, MyFootprints:SD_ESD, symbol SD_ESD:TPD1E05U06DPYR
- added D10, D11, D6, D7: BAT54S, MyFootprints:dual_shottkey, symbol dual_shottkey:BAT54S
- added H1, H2, H3, H4: MountingHole, MountingHole:MountingHole_3.2mm_M3, symbol Mechanical:MountingHole
- added J10, J9: Conn_01x03, Connector_Wire:SolderWire-0.5sqmm_1x03_P4.6mm_D0.9mm_OD2.1mm_Relief, symbol Connector_Generic:Conn_01x03
- added J15: Conn_01x08, Connector_PinSocket_2.54mm:PinSocket_1x08_P2.54mm_Vertical, symbol Connector_Generic:Conn_01x08
- added J3: UART1, Connector_PinSocket_2.54mm:PinSocket_1x04_P2.54mm_Vertical, symbol Connector_Generic:Conn_01x04
- added J4: UART3, Connector_PinSocket_2.54mm:PinSocket_1x04_P2.54mm_Vertical, symbol Connector_Generic:Conn_01x04
- added J8: MEM2061-01-188-00-A_REVA, MyFootprints:SD_Card, symbol SD_Card:MEM2061-01-188-00-A_REVA
- added R16, R17, R18, R19, R20, R21: 22, Resistor_SMD:R_0402_1005Metric, symbol Device:R
- added R22, R23, R24, R27, R32, R33: 47k, Resistor_SMD:R_0402_1005Metric, symbol Device:R
- added R25, R26, R34, R41: 20, Resistor_SMD:R_1206_3216Metric, symbol Device:R_Small
- added R28, R29, R35, R42: 130, Resistor_SMD:R_0805_2012Metric, symbol Device:R_Small
- added R30, R31, R36, R43: 4.7k, Resistor_SMD:R_0402_1005Metric, symbol Device:R
- added R52, R53, R54, R55, R56, R57, R58, R59, R60: 100, Resistor_SMD:R_0402_1005Metric, symbol Device:R
- SW2: value PTS526 SM15 SMTR2 LFS -> BOOT
- gave numbers to parts that had none: 39
Connections:
- net AGND is gone; now on net GND: C17.2
- net PGND is gone; now on net GND: CR3.2, J6.A1_B12 (GND), J6.B1_A12 (GND__1), J6.SH1 (SHELL_GND), J6.SH2 (SHELL_GND__1), J6.SH3 (SHELL_GND__2), J6.SH4 (SHELL_GND__3)
- net 15V0: now also J10.1 (Pin_1), J15.5 (Pin_5), J9.1 (Pin_1)
- net 3V3: now also C43.1, C44.1, C69.2, C70.2, C71.2, D10.2, D11.2, D13.1 (I/O), D16.1 (I/O), D20.1 (I/O), D6.2, D7.2, J15.8 (Pin_8), J3.4 (Pin_4), J4.4 (Pin_4), J8.4 (VDD), R22.1, R23.2, R24.1, R27.1, R32.1, R33.1
- net 3V3_BUCK: now also C30.1, R11.1, U4.6 (IN2); no longer C29.2, R10.2, U4.8 (IN1)
- net 3V3_LDO: now also C29.2, R10.2, U4.8 (IN1); no longer C30.1, R11.1, U4.6 (IN2)
- net CLK: now also R58.2
- net CS1: now also U3.21 (PA5)
- net CS2: now also U3.22 (PA6)
- net CS3: now also U3.23 (PA7)
- net CS4: now also U3.24 (PC4)
- net GND: now also U5.9 (Thermal_Pad), C43.2, C44.2, C45.2, C46.2, C47.2, C68.2, C69.1, C70.1, C71.1, CR6.1, CR7.1, CR8.1, CR9.1, D1.2 (GND), D10.1, D11.1, D12.2 (GND), D13.2 (GND), D14.2 (GND), D15.2 (GND), D16.2 (GND), D17.2 (GND), D18.2 (GND), D19.2 (GND), D2.2 (GND), D20.2 (GND), D21.2 (GND), D22.2 (GND), D23.2 (GND), D3.2 (GND), D4.2 (GND), D5.2 (GND), D6.1, D7.1, D8.2 (GND), D9.2 (GND), J10.2 (Pin_2), J15.1 (Pin_1), J3.1 (Pin_1), J4.1 (Pin_1), J8.11 (GND), J8.12 (GND__1), J8.6 (VSS), J8.9 (CD1), J9.2 (Pin_2), R28.1, R29.1, R35.1, R42.1
- net MISO: now also R56.2
- net MOSI: now also R57.2; no longer U3.53 (PC12)
- net NRST: now also C26.2, R9.2, SW1.1, SW1.2
- net RX1: now also R52.2
- net RX3: now also R54.2
- net TX1: now also R53.2
- net TX3: now also R55.2
- net SW: now reaches C15.2, L1.1, U1.12 (SW), U1.3 (NC)
- net P2: now reaches U3.10 (PC2)
- net P2: now also C68.1, D11.3, R43.2
- net P3: now reaches U3.11 (PC3)
- net P3: now also C46.1, D7.3, R31.2
- net GPIO_OUT_1: now reaches U3.25 (PC5)
- net GPIO_OUT_1: now also R60.2
- net GPIO_OUT_0: now reaches U3.26 (PB0)
- net GPIO_OUT_0: now also R59.2
- net SD_DET: now reaches U3.38 (PC7)
- net SD_DET: now also D2.1 (I/O), J8.10 (CD2), R23.1
- net SD_D0: now reaches U3.39 (PC8)
- net SD_D0: now also D3.1 (I/O), R16.1, R24.2
- net SD_D1: now reaches U3.40 (PC9)
- net SD_D1: now also D4.1 (I/O), R17.1, R27.2
- net P0: now reaches U3.8 (PC0)
- net P0: now also C45.1, D6.3, R30.2
- net P1: now reaches U3.9 (PC1)
- net P1: now also C47.1, D10.3, R36.2
- net SW1: now reaches C16.2, L2.1, U2.12 (SW), U2.3 (NC)
- net BAT_FUSE: now reaches CR1.2, F1.2
- net BAT_IN: now reaches F1.1, J1.2 (Pin_2)
- net CLK3 renamed SD_D2
- net SD_D2: now also D8.1 (I/O), R18.1, R32.2
- net CS_SD renamed SD_CMD
- net SD_CMD: now also D1.1 (I/O), R20.1, R22.2
- net MISO3 renamed SD_D3
- net SD_D3: now also D9.1 (I/O), R19.1, R33.2
- net Pressure_3: no longer names the net of J5.3 (Pin_3)
- net Pressure_3: now also R26.2
- net Pressure_4: no longer names the net of J7.3 (Pin_3)
- net Pressure_4: now also R25.2
- new net: D23.1 (I/O), J15.7 (Pin_7), R60.1
- new net: D12.1 (I/O), J3.2 (Pin_2), R52.1
- new net: D14.1 (I/O), J3.3 (Pin_3), R53.1
- new net: D19.1 (I/O), J15.2 (Pin_2), R57.1
- new net: D21.1 (I/O), J15.4 (Pin_4), R58.1
- new net: D17.1 (I/O), J4.2 (Pin_2), R55.1
- new net: CR8.2, R34.1, R35.2, R36.1
- new net: J9.3 (Pin_3), R34.2
- new net: J8.3 (CMD), R20.2
- new net: CR9.2, R41.1, R42.2, R43.1
- new net: CR7.2, R26.1, R29.2, R31.1
- new net: D15.1 (I/O), J4.3 (Pin_3), R54.1
- new net: J8.1 (DAT2), R18.2
- new net: CR6.2, R25.1, R28.2, R30.1
- new net: J8.7 (DAT0), R16.2
- new net: J8.2 (CD/DAT3), R19.2
- new net: D22.1 (I/O), J15.6 (Pin_6), R59.1
- new net: D18.1 (I/O), J15.3 (Pin_3), R56.1
- new net: J10.3 (Pin_3), R41.2
- new net: J8.8 (DAT1), R17.2
- new net: J8.5 (CLK), R21.2
- new net SD_CLK: D5.1 (I/O), R21.1, U3.53 (PC12)
- no-connect marks 16 -> 35
Other:
- note added: "Breakout Periferals"
- note added: "SD CARD"
- moved on the sheet: C33, C34, C48, C49, C50, C51, C52, C53, C54, C55, C56, C57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

Commit message: order read
Parts:
- added LED5: LTST-C190KRKT, MyFootprints:red_LED, symbol red_led:LTST-C190KRKT
- added R61: 130, Resistor_SMD:R_0805_2012Metric, symbol Device:R_Small
Connections:
- net GND: now also LED5.1
- net STATUS_LED: now reaches U3.27 (PB1)
- net STATUS_LED: now also R61.2
- new net: LED5.2, R61.1
- no-connect marks 35 -> 34
Other:
- moved on the sheet: C43

Commit message: reworked power poath, added cs multiplexer
Parts:
- removed CR2: SMBJ28A-13-F, MyFootprints:28V_TVS, symbol 28V_TVS:SMBJ28A-13-F
- removed J10, J5, J7, J9: Conn_01x03, Connector_Wire:SolderWire-0.5sqmm_1x03_P4.6mm_D0.9mm_OD2.1mm_Relief, symbol Connector_Generic:Conn_01x03
- removed L1, L2: XAL4040-153MEC, MyFootprints:15uH_Inductor, symbol 15uH_Inductor:XAL4040-153MEC
- removed U2: LMR36006CRNXT, MyFootprints:15V_Buck, symbol 15V_Buck:LMR36006CRNXT
- added C72, C73, C77: 4.7u, Capacitor_SMD:C_1206_3216Metric, symbol Device:C
- added C74, C75, C76, C78, C79: 0.1u, Capacitor_SMD:C_0402_1005Metric, symbol Device:C
- added C80: 1u, Capacitor_SMD:C_0603_1608Metric, symbol Device:C
- added D24: SMBJ15A, MyFootprints:15V_TVS, symbol 15V_TVS:SMBJ15A
- added D25: SMBJ18A, MyFootprints:18V_TVS, symbol 18V_TVS:SMBJ18A
- added D26, D27, D28, D29, D30, D31, D32, D33, D34, D35, D36: TPD1E05U06DPYR, MyFootprints:SD_ESD, symbol SD_ESD:TPD1E05U06DPYR
- added J10, J5, J7, J9: SM03B-GHS-TB, MyFootprints:3-pin-jst, symbol 3-pin-jst:SM03B-GHS-TB
- added J16: C36191, Connector_PinSocket_2.54mm:PinSocket_2x06_P2.54mm_Vertical, symbol Connector_Generic:Conn_02x06_Odd_Even
- added L1, L2: IHLP2525CZER220M5A, MyFootprints:22uH, symbol 22uH:IHLP2525CZER220M5A
- added LED6: LTST-C190KRKT, MyFootprints:red_LED, symbol red_led:LTST-C190KRKT
- added R62, R64: 68.1k, Resistor_SMD:R_0402_1005Metric, symbol Device:R
- added R63, R69, R72, R75, R76, R77, R78: 10k, Resistor_SMD:R_0402_1005Metric, symbol Device:R
- added R65, R66, R74: 100k, Resistor_SMD:R_0402_1005Metric, symbol Device:R
- added R67, R70, R73: 4.7k, Resistor_SMD:R_0402_1005Metric, symbol Device:R
- added R68: 590, Resistor_SMD:R_0402_1005Metric, symbol Device:R
- added R71, R79, R91, R92: 130, Resistor_SMD:R_0805_2012Metric, symbol Device:R_Small
- added R80, R81, R82, R83, R84, R85, R86, R87, R88, R89, R90: 100, Resistor_SMD:R_0402_1005Metric, symbol Device:R
- added U10: SS34, MyFootprints:Boost_Shottkey, symbol Boost_Shottkey:SS34
- added U11: CD74HC154M96, MyFootprints:4-16-Multiplexer, symbol 4-16-Multiplexer:CD74HC154M96
- added U12: TPS26600PWPR, MyFootprints:eFuse, symbol eFuse:TPS26600PWPR
- added U2: TPS55340PWPR, MyFootprints:15V_Boost, symbol 15V_Boost:TPS55340PWPR
- C10: value 220n -> 10n; footprint Capacitor_SMD:C_0805_2012Metric -> Capacitor_SMD:C_0402_1005Metric
- C13: value 1u -> 270n; footprint Capacitor_SMD:C_0603_1608Metric -> Capacitor_SMD:C_0402_1005Metric
- C16: value 0.1u -> 100p
- C18: value CFF -> 0.1u; footprint Capacitor_SMD:C_0603_1608Metric -> Capacitor_SMD:C_0402_1005Metric; now fitted
- C20: value 0.1u -> 4.7u; footprint Capacitor_SMD:C_0402_1005Metric -> Capacitor_SMD:C_1206_3216Metric
- C22, C24: value 10u -> 4.7u; footprint Capacitor_SMD:C_1210_3225Metric -> Capacitor_SMD:C_1206_3216Metric
- C9: value 220n -> 0.1u; footprint Capacitor_SMD:C_0805_2012Metric -> Capacitor_SMD:C_0402_1005Metric
- J1: footprint Connector_Wire:SolderWire-0.5sqmm_1x02_P4.6mm_D0.9mm_OD2.1mm_Relief -> Connector_AMASS:AMASS_XT60-F_1x02_P7.20mm_Vertical
- R2: value 100k -> 590
- R5: value 7.15k -> 43.2k
- R7: value 43.2k -> 24.9k
- U3: value STM32L496RGT6 -> STM32L496RET6
Connections:
- net SW1 is gone; now on net GND: C16.2
- net 15V0: now also C76.1, C77.1, D25.1 (K), J10.1, J5.1, J7.1, J9.1, U12.15 (OUT), U12.16 (OUT); no longer C18.1, C20.1, C22.1, C24.1, R2.1
- net 3V3: now also C17.1, R1.2, U5.1 (OUT), C79.2, C80.2, R74.2, R75.1, R76.1, R77.1, R78.1, U11.24 (VCC); no longer C31.1, C32.1, R15.2, U4.7 (OUT)
- net 5V0: now also C31.1, C32.1, U4.7 (OUT), R79.2; no longer C1.2, C11.1, C4.1, CR3.5, J6.A4_B9 (VBUS), J6.B4_A9 (VBUS__1)
- net CLK: now also R57.2; no longer R58.2
- net CS1: now also R38.2, U7.9 (*CS), U11.2 (*Y1); no longer R37.2, U3.21 (PA5), U6.9 (*CS)
- net CS2: now also R39.2, U8.9 (*CS), U11.3 (*Y2); no longer R38.2, U3.22 (PA6), U7.9 (*CS)
- net CS3: now also R40.2, U9.9 (*CS), U11.4 (*Y3); no longer R39.2, U3.23 (PA7), U8.9 (*CS)
- net CS4: now also R80.1, U11.5 (*Y4); no longer R40.2, U3.24 (PC4), U9.9 (*CS)
- net GND: now also C10.2, C18.2, C9.2, C72.2, C73.2, C74.2, C75.1, C76.2, C77.2, C78.2, C79.1, C80.1, D24.2 (A), D25.2 (A), D26.2 (GND), D27.2 (GND), D28.2 (GND), D29.2 (GND), D30.2 (GND), D31.2 (GND), D32.2 (GND), D33.2 (GND), D34.2 (GND), D35.2 (GND), D36.2 (GND), J10.2, J16.12 (Pin_12), J5.2, J7.2, J9.2, LED6.1, R63.2, R64.2, R70.1, R73.1, U11.12 (GND), U11.18 (*E1), U11.19 (*E2), U12.17 (PAD), U12.6 (MODE), U12.8 (RTN), U12.9 (GND), U2.11 (NC), U2.12 (PGND), U2.13 (PGND), U2.14 (PGND), U2.15 (EPAD), U2.6 (SYNC), U2.7 (AGND); no longer C10.1, C9.1, R5.2
- net MOSI: now also R58.2; no longer R57.2
- net RX1: now also R53.2; no longer R52.2
- net RX3: now also R55.2; no longer R54.2
- net SW: now also L2.2
- net TX1: now also R52.2; no longer R53.2
- net TX3: now also R54.2; no longer R55.2
- net VBAT: now also C9.1, D24.1 (K), L1.2, U2.3 (VIN), U2.4 (EN); no longer C10.2, C9.2
- net at R34.2: now also J9.3
- net at C13.1: now also R2.2
- net at R25.2: now also J5.3
- net at R26.2: now also J7.3
- net at R41.2: now also J10.3
- net at C16.1: now also R2.1, U2.8 (COMP)
- net 3V3_BUCK renamed 5V_BUCK
- net 5V_BUCK: now also C29.2, R10.2, U4.8 (IN1), L2.1, R71.2; no longer C30.1, R11.1, R14.2, U4.6 (IN2)
- removed net 3V3_LDO: C17.1, C29.2, R1.2, R10.2, U4.8 (IN1), U5.1 (OUT)
- new net: C78.1, R74.1, U12.7 (SHDN_N)
- new net: R14.2, R71.1
- new net: R65.2, R66.1
- new net: R66.2, R67.2, U12.3 (UVLO)
- new net: R64.1, U2.10 (FREQ)
- new net: R5.2, R62.1
- new net: R67.1, R68.1
- new net: R15.2, R79.1
- new net: R72.1, U12.11 (ILIM)
- new net: R72.2, R73.2
- new net: C75.2, U12.12 (DVDT)
- new net: LED6.2, R92.1
- new net: R68.2, R69.1, U12.5 (OVP)
- new net: R69.2, R70.2
- new net: R91.1, R92.2
- new net: C10.1, U2.5 (SS)
- new net: R62.2, R63.1, U2.9 (FB)
- new net 15V0_Boost: C18.1, C20.1, C22.1, C24.1, C72.1, C73.1, C74.1, R5.1, R65.1, U10.1 (CATHODE), U12.1 (IN), U12.2 (IN)
- new net 5V_USB: C1.2, C11.1, C30.1, C4.1, CR3.5, J6.A4_B9 (VBUS), J6.B4_A9 (VBUS__1), R11.1, R91.2, U4.6 (IN2)
- new net A0: R75.2, U11.23 (A0), U3.21 (PA5)
- new net A1: R77.2, U11.22 (A1), U3.22 (PA6)
- new net A2: R78.2, U11.21 (A2), U3.23 (PA7)
- new net A3: R76.2, U11.20 (A3), U3.24 (PC4)
- new net ANODE: L1.1, U10.2 (ANODE), U2.1 (SW), U2.2 (SW)
- new net CS0: R37.2, U11.1 (*Y0), U6.9 (*CS)
- new net CS10: R90.1, U11.11 (*Y10)
- new net CS11: R89.1, U11.13 (*Y11)
- new net CS12: R88.1, U11.14 (*Y12)
- new net CS13: R87.1, U11.15 (*Y13)
- new net CS14: R86.1, U11.16 (*Y14)
- new net CS5: R81.1, U11.6 (*Y5)
- new net CS6: R82.1, U11.7 (*Y6)
- new net CS7: R83.1, U11.8 (*Y7)
- new net CS8: R84.1, U11.9 (*Y8)
- new net CS9: R85.1, U11.10 (*Y9)
- new net S1: D29.1 (I/O), J16.1 (Pin_1), R80.2
- new net S10: D36.1 (I/O), J16.8 (Pin_8), R89.2
- new net S11: D27.1 (I/O), J16.10 (Pin_10), R90.2
- new net S2: D31.1 (I/O), J16.3 (Pin_3), R81.2
- new net S3: D33.1 (I/O), J16.5 (Pin_5), R82.2
- new net S4: D35.1 (I/O), J16.7 (Pin_7), R83.2
- new net S5: D26.1 (I/O), J16.9 (Pin_9), R84.2
- new net S6: D28.1 (I/O), J16.11 (Pin_11), R85.2
- new net S7: D30.1 (I/O), J16.2 (Pin_2), R86.2
- new net S8: D32.1 (I/O), J16.4 (Pin_4), R87.2
- new net S9: D34.1 (I/O), J16.6 (Pin_6), R88.2
- no-connect marks 34 -> 38
Other:
- note added: "SPI"
- note added: "SPI CS"
- note added: "UART1"
- note added: "UART2"
- moved on the sheet: C1, C11, C14, C17, C26, C33, C34, C35, C36, C37, C38, C39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

Commit message: prod ready
Parts:
- C69, C70, C71: value 10u -> 1u; footprint Capacitor_SMD:C_1210_3225Metric -> Capacitor_SMD:C_0603_1608Metric
- J1: footprint Connector_AMASS:AMASS_XT60-F_1x02_P7.20mm_Vertical -> Connector_AMASS:AMASS_XT60-M_1x02_P7.20mm_Vertical
